File: GPS_Tracker/Transmitter.sch (KiCad schematic (older format))
At the start: 0 parts

Commit message: added circuits
Parts:
- added AE?: Antenna, symbol Device:Antenna
- added C?: 100pF, symbol pspice:CAP
- added C?: 1.0uF, symbol pspice:CAP
- added U?: XBee_SMT, RF_Module:Digi_XBee_SMT, symbol RF_ZigBee:XBee_SMT
Connections:
- new net: C?.1, U?.2 (VCC)
- new net: AE?.1 (A), U?.36 (RF)
- new net +3V3: C?.1
- new net GND: C?.2, C?.2, U?.1 (GND), U?.11 (GND), U?.13 (GND), U?.22 (GND), U?.35 (GND)
- new net Trans_RX: U?.4 (DIO14/UART_RX/~CONFIG)
- new net Trans_TX: U?.3 (DIO13/UART_TX)
Changed lines of the file:
@@
 $Descr A4 11693 8268
 encoding utf-8
-Sheet 1 6
+Sheet 1 1
 Title ""
 Date ""
@@
 Comment4 ""
 $EndDescr
+$Comp
+L RF_ZigBee:XBee_SMT U?
+U 1 1 5E6E6EA9
+P 5150 4250
+F 0 "U?" H 5150 5431 50  0000 C CNN
+F 1 "XBee_SMT" H 5150 5340 50  0000 C CNN
+F 2 "RF_Module:Digi_XBee_SMT" H 5990 3190 50  0001 C CNN
+F 3 "http://www.digi.com/resources/documentation/digidocs/pdfs/90002126.pdf" H 5150 3850 50  0001 C CNN
+	1    5150 4250
+	1    0    0    -1
+$EndComp
+$Comp
+L power:GND #PWR?
+U 1 1 5E6E8515
+P 5150 5850
+F 0 "#PWR?" H 5150 5600 50  0001 C CNN
+F 1 "GND" H 5155 5677 50  0000 C CNN
+F 2 "" H 5150 5850 50  0001 C CNN
+F 3 "" H 5150 5850 50  0001 C CNN
+	1    5150 5850
+	1    0    0    -1
+$EndComp
+Wire Wire Line
+	4950 5350 4950 5850
+Wire Wire Line
+	5150 5850 5250 5850
+Wire Wire Line
+	5350 5850 5350 5350
+Connection ~ 5150 5850
+Wire Wire Line
+	5050 5350 5050 5850
+Wire Wire Line
+	4950 5850 5050 5850
+Connection ~ 5050 5850
+Wire Wire Line
+	5050 5850 5150 5850
+Wire Wire Line
+	5150 5350 5150 5850
+Wire Wire Line
+	5250 5350 5250 5850
+Connection ~ 5250 5850
+Wire Wire Line
+	5250 5850 5350 5850
+$Comp
+L Device:Antenna AE?
+U 1 1 5E6E9567
+P 7200 4000
+F 0 "AE?" H 7280 3989 50  0000 L CNN
+F 1 "Antenna" H 7280 3898 50  0000 L CNN
+F 2 "" H 7200 4000 50  0001 C CNN
+F 3 "~" H 7200 4000 50  0001 C CNN
+	1    7200 4000
+	1    0    0    -1
+$EndComp
+Wire Wire Line
+	6250 4250 7200 4250
+Wire Wire Line
+	7200 4250 7200 4200
+$Comp
+L pspice:CAP C?
+U 1 1 5E6EA76B
+P 6750 2300
+F 0 "C?" H 6928 2346 50  0000 L CNN
+F 1 "100pF" H 6928 2255 50  0000 L CNN
+F 2 "" H 6750 2300 50  0001 C CNN
+F 3 "~" H 6750 2300 50  0001 C CNN
+	1    6750 2300
+	1    0    0    -1
+$EndComp
+$Comp
+L pspice:CAP C?
+U 1 1 5E6EAB35
+P 7450 2300
+F 0 "C?" H 7628 2346 50  0000 L CNN
+F 1 "1.0uF" H 7628 2255 50  0000 L CNN
+F 2 "" H 7450 2300 50  0001 C CNN
+F 3 "~" H 7450 2300 50  0001 C CNN
+	1    7450 2300
+	1    0    0    -1
+$EndComp
+$Comp
+L power:GND #PWR?
+U 1 1 5E6EAE7D
+P 7050 2700
+F 0 "#PWR?" H 7050 2450 50  0001 C CNN
+F 1 "GND" H 7055 2527 50  0000 C CNN
+F 2 "" H 7050 2700 50  0001 C CNN
+F 3 "" H 7050 2700 50  0001 C CNN
+	1    7050 2700
+	1    0    0    -1
+$EndComp
+$Comp
+L power:+3.3V #PWR?
+U 1 1 5E6EB4B8
+P 7450 1700
+F 0 "#PWR?" H 7450 1550 50  0001 C CNN
+F 1 "+3.3V" H 7465 1873 50  0000 C CNN
+F 2 "" H 7450 1700 50  0001 C CNN
+F 3 "" H 7450 1700 50  0001 C CNN
+	1    7450 1700
+	1    0    0    -1
+$EndComp
+Wire Wire Line
+	6750 2550 6750 2700
+Wire Wire Line
+	6750 2700 7050 2700
+Wire Wire Line
+	7050 2700 7450 2700
+Wire Wire Line
+	7450 2700 7450 2550
+Connection ~ 7050 2700
+Wire Wire Line
+	7450 2050 7450 1700
+Wire Wire Line
+	6750 2050 5150 2050
+Wire Wire Line
+	5150 2050 5150 3250
+Text GLabel 3700 3450 0    50   Input ~ 0
+Trans_TX
+Text GLabel 3700 3550 0    50   Input ~ 0
+Trans_RX
+Wire Wire Line
+	4050 3450 3700 3450
+Wire Wire Line
+	4050 3550 3700 3550
 $EndSCHEMATC
