File: Mini_GPS_Tracker/Mini_GPS_Tracker.kicad_pcb (KiCad board)
At the start: 2 copper layers, 38.1 x 99.1 mm, 54 parts, among them J1 USB_C_Receptacle, J2 Screw_Terminal_01x02, J3 901-10512-1, J4 Conn_ARM_JTAG_SWD_10, SW1 SW_Push, SW2 MLL1200S, U1 CH340E, U2 MS5611-01BA, U3 LD1117S33TR_SOT223, U4 MAX-8Q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

Commit message: added routing
Parts:
- added LS1: CSS-J4D20-SMT, Sparkfun-Artemis:CUI_CSS-J4D20-SMT, F.Cu at (153.0, 53.4)
- added R7: R, Resistor_SMD:R_0805_2012Metric_Pad1.15x1.40mm_HandSolder, F.Cu at (152.9, 59.9)
- moved FB2 16.8 mm to (160.7, 107.7), turned to 0 degrees
- moved FB1 12.4 mm to (160.4, 111.3), turned to 0 degrees
- moved D4 5.04 mm to (148.7, 121.5), turned to 270 degrees
- moved C13 4.38 mm to (153.2, 64.9)
- moved C12 4.38 mm to (153.2, 62.7)
- moved C14 4.38 mm to (153.2, 67.1)
- moved C15 4.38 mm to (153.2, 69.3)
- moved C16 4.38 mm to (153.2, 71.6)
- moved C17 4.38 mm to (153.2, 76.3)
- moved C18 4.38 mm to (153.2, 74.0)
- moved U7 4.38 mm to (152.8, 81.3), turned to 0 degrees
- moved R6 4.15 mm to (152.8, 121.7), turned to 270 degrees
- moved J4 3.22 mm to (170.4, 86.1), turned to 270 degrees
- moved D1 1.49 mm to (165.4, 116.1)
- moved D2 1.49 mm to (165.4, 122.6)
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Connections:
- MD1 pad 16: Net-(MD1-Pad16) -> buzzer
Routing:
- net GND: track 0.00 -> 369.7 mm, vias 0 -> 11
- net +3V3: track 0.00 -> 127.3 mm, vias 0 -> 7
- net RTS: track 0.00 -> 37.4 mm, vias 0 -> 2
- net gps_reset: track 0.00 -> 30.8 mm, vias 0 -> 2
- net RESET: track 0.00 -> 26.9 mm, vias 0 -> 3
- net MOSI_Flash: track 0.00 -> 25.0 mm
- net Net-(J3-Pad1): track 0.00 -> 20.9 mm
- net Net-(C9-Pad1): track 0.00 -> 19.4 mm
- net Pressure_SDA: track 0.00 -> 18.3 mm, vias 0 -> 2
- net Net-(LS1-PadP1): track 0.00 -> 18.1 mm
- net MISO_Flash: track 0.00 -> 17.8 mm, vias 0 -> 2
- net Net-(FB2-Pad1): track 0.00 -> 15.0 mm
- net Pressure_SCL: track 0.00 -> 12.7 mm, vias 0 -> 2
- net SWDCK: track 0.00 -> 12.0 mm, vias 0 -> 2
- net Net-(FB1-Pad1): track 0.00 -> 11.8 mm
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
Commit message: updated routing
Routing:
- net buzzer: track 2.74 -> 67.2 mm, vias 1 -> 4
- net TRANS_TX: track 3.99 -> 52.9 mm
- net +3V3: track 127.3 -> 174.0 mm, vias 7 -> 12
- net GND: track 369.7 -> 412.3 mm, vias 11 -> 14
- net TRANS_RX: track 4.10 -> 44.5 mm
- net 9_SDA: track 0.00 -> 27.2 mm, vias 0 -> 4
- net v_measure: track 4.23 -> 27.7 mm, vias 1 -> 2
- net GPS_RX: track 0.00 -> 22.1 mm, vias 0 -> 2
- net clk_flash: track 1.99 -> 21.7 mm, vias 1 -> 2
- net 9_SCL: track 0.00 -> 18.0 mm, vias 0 -> 3
- net RESET: track 26.9 -> 40.6 mm
- net Net-(C18-Pad1): track 0.00 -> 6.90 mm
- net GPS_TX: track 2.33 -> 9.15 mm
- net Net-(C2-Pad1): track 1.47 -> 8.06 mm, vias 1 -> 2
- net Net-(C17-Pad1): track 0.00 -> 4.08 mm
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
Commit message: trying to do a 4 layer pcb
Routing:
- net GND: track 412.3 -> 23.4 mm, vias 14 -> 0
- net +3V3: track 174.0 -> 5.75 mm, vias 12 -> 0
- net buzzer: track 67.2 -> 1.50 mm, vias 4 -> 0
- net gps_reset: track 30.8 -> 0.10 mm, vias 2 -> 0
- net 9_SDA: track 27.2 -> 0.00 mm, vias 4 -> 0
- net v_measure: track 27.7 -> 2.27 mm, vias 2 -> 0
- net A1: track 3.29 -> 28.6 mm
- net MOSI_Flash: track 25.0 -> 0.80 mm
- net GPS_RX: track 22.1 -> 0.10 mm, vias 2 -> 0
- net clk_flash: track 21.7 -> 0.00 mm, vias 2 -> 0
- net Net-(J3-Pad1): track 20.9 -> 0.00 mm
- net RESET: track 40.6 -> 21.2 mm, vias 3 -> 2
- net 9_SCL: track 18.0 -> 0.00 mm, vias 3 -> 0
- net MISO_Flash: track 17.8 -> 0.10 mm, vias 2 -> 0
- net SWDCK: track 14.0 -> 1.88 mm, vias 2 -> 1
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- added copper zone on PWR, net +3V3
- added copper zone on GND, net GND
Other:
- copper layers 2 -> 4
