File: Mini_GPS_Tracker/Mini_GPS_Tracker.kicad_pcb (KiCad board)
At the start: 4 copper layers, 38.1 x 105.4 mm, 62 parts, among them J1 USB_C_Receptacle, J2 Screw_Terminal_01x02, J3 901-10512-1, J4 Conn_ARM_JTAG_SWD_10, SW1 SW_Push, SW2 MLL1200S, U1 FT230XS, U10 STMICROELECTRONICS_STM32H747X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, U11 ADXL343, U12 BNO055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

Commit message: updated core
Parts:
- added C15: 0.1uF, Capacitor_SMD:C_0805_2012Metric_Pad1.15x1.40mm_HandSolder, F.Cu at (264.8, 37.9)
- added C16: 0.1uF, Capacitor_SMD:C_0805_2012Metric_Pad1.15x1.40mm_HandSolder, F.Cu at (264.8, 40.9)
- added C17: 22pF, Capacitor_SMD:C_0805_2012Metric_Pad1.15x1.40mm_HandSolder, F.Cu at (269.5, 37.9)
- added C18: 22pF, Capacitor_SMD:C_0805_2012Metric_Pad1.15x1.40mm_HandSolder, F.Cu at (264.8, 43.8)
- added MD1: SPARKFUN_WRL-15376, Sparkfun-Artemis:SPARKFUN_WRL-15376, F.Cu at (166.4, 149.7)
- added R4: 10K, Resistor_SMD:R_0805_2012Metric_Pad1.15x1.40mm_HandSolder, F.Cu at (269.5, 40.9)
- added R5: 10k, Resistor_SMD:R_0805_2012Metric_Pad1.15x1.40mm_HandSolder, F.Cu at (274.3, 37.9)
- added R8: 10k, Resistor_SMD:R_0805_2012Metric_Pad1.15x1.40mm_HandSolder, F.Cu at (269.5, 43.8)
- added U11: STM32F413ZHTx, Package_QFP:LQFP-144_20x20mm_P0.5mm, F.Cu at (224.0, 48.6)
- added Y2: 32.7568KHz, Crystal:Crystal_SMD_2012-2Pin_2.0x1.2mm_HandSoldering, F.Cu at (274.1, 40.8)
- U10: value STMICROELECTRONICS_STM32H747XIH6 -> LBEE5KL1DX-TEMP; footprint Package_BGA:TFBGA-265_14x14mm_Layout17x17_P0.8mm -> Sparkfun-Artemis:XCVR_LBEE5KL1DX-TEMP
- moved U10 59.0 mm to (265.9, 53.3)
- renumbered C23 to C14, C8 to C3, C21 to C5, C22 to C8, U11 to U1, U12 to U7
Connections:
- net Net-(U12-Pad11) renamed /Sheet5E70BD5D/BNO055_RESET
- net Net-(U12-Pad14) renamed /Sheet5E70BD5D/BNO055_INTERRUPT
- net Net-(U12-Pad19) renamed /Sheet5E70BD5D/BNO055_SCL
- net Net-(U12-Pad20) renamed /Sheet5E70BD5D/BNO055_SDA
- U7 pad 10: Net-(U12-Pad10) -> GND
- U7 pad 12: Net-(U12-Pad12) -> Net-(U7-Pad12)
- U7 pad 13: Net-(U12-Pad13) -> Net-(U7-Pad13)
- U7 pad 15: Net-(U12-Pad15) -> GND
- U7 pad 16: Net-(U12-Pad15) -> GND
- U7 pad 18: Net-(U12-Pad18) -> GND
- U7 pad 2: Net-(U12-Pad2) -> GND
- U7 pad 25: Net-(U12-Pad15) -> GND
- U7 pad 26: Net-(U12-Pad26) -> Net-(C17-Pad1)
- U7 pad 28: Net-(U12-Pad28) -> +3V3
- U7 pad 3: Net-(U12-Pad3) -> +3V3
- U7 pad 4: Net-(U12-Pad4) -> +3V3
