File: Mini_GPS_Tracker/GPS.sch (KiCad schematic (older format))
At the start: 12 parts, among them U4 MAX-8Q, U5 SGGP.12.4.A.02, U9 MAX2686

Commit message: Adding BNO055 Motion co-processor
Parts:
- U5: symbol Sparkfun~Artemis:SGGP.12.4.A.02 -> Mini_GPS_Tracker-rescue:SGGP.12.4.A.02-Sparkfun_Artemis
- U9: symbol Sparkfun~Artemis:MAX2686 -> Mini_GPS_Tracker-rescue:MAX2686-Sparkfun_Artemis
Changed lines of the file:
@@
 EESchema Schematic File Version 4
+LIBS:Mini_GPS_Tracker-cache
 EELAYER 30 0
 EELAYER END
 $Descr A4 11693 8268
 encoding utf-8
-Sheet 4 6
+Sheet 4 7
 Title ""
 Date ""
@@
 	3700 3900 3750 3900
 $Comp
-L Sparkfun~Artemis:SGGP.12.4.A.02 U5
+L Mini_GPS_Tracker-rescue:SGGP.12.4.A.02-Sparkfun_Artemis U5
 U 1 1 5E7667EA
 P 7850 1850
@@
 $EndComp
 $Comp
-L Sparkfun~Artemis:MAX2686 U9
+L Mini_GPS_Tracker-rescue:MAX2686-Sparkfun_Artemis U9
 U 1 1 5E78E34D
 P 7850 4600
