File: Mini_GPS_Tracker/GPS.sch (KiCad schematic (older format))
At the start: 5 parts, among them U3 MAX-8Q

Commit message: updates to routing
Parts:
- FB1, FB2: footprint (none) -> Capacitor_SMD:C_0805_2012Metric_Pad1.15x1.40mm_HandSolder
Connections:
- wire segments 18 -> 20
Changed lines of the file:
@@
 	1    0    0    -1
 $EndComp
-Wire Wire Line
-	6700 3100 6800 3100
-Wire Wire Line
-	6700 3100 6700 3450
 $Comp
 L Device:Ferrite_Bead_Small FB1
@@
 F 0 "FB1" V 4763 3050 50  0000 C CNN
 F 1 "Ferrite_Bead_Small" V 4854 3050 50  0000 C CNN
-F 2 "" V 4930 3050 50  0001 C CNN
+F 2 "Capacitor_SMD:C_0805_2012Metric_Pad1.15x1.40mm_HandSolder" V 4930 3050 50  0001 C CNN
 F 3 "~" H 5000 3050 50  0001 C CNN
 	1    5000 3050
@@
 F 0 "FB2" V 4763 3150 50  0000 C CNN
 F 1 "Ferrite_Bead_Small" V 4854 3150 50  0000 C CNN
-F 2 "" V 4930 3150 50  0001 C CNN
+F 2 "Capacitor_SMD:C_0805_2012Metric_Pad1.15x1.40mm_HandSolder" V 4930 3150 50  0001 C CNN
 F 3 "~" H 5000 3150 50  0001 C CNN
 	1    5000 3150
@@
 Wire Wire Line
 	5100 3050 5150 3050
+Wire Wire Line
+	6700 3450 6700 3300
+Wire Wire Line
+	6700 3300 6800 3300
+$Comp
+L power:GND #PWR0122
+U 1 1 5E7583F9
+P 6600 3200
+F 0 "#PWR0122" H 6600 2950 50  0001 C CNN
+F 1 "GND" H 6605 3027 50  0000 C CNN
+F 2 "" H 6600 3200 50  0001 C CNN
+F 3 "" H 6600 3200 50  0001 C CNN
+	1    6600 3200
+	1    0    0    -1
+$EndComp
+Wire Wire Line
+	6600 3200 6600 3100
+Wire Wire Line
+	6600 3100 6800 3100
 $EndSCHEMATC

Commit message: updated antenna;
Parts:
- removed AE1: CGGBP.35.6.A.02, Sparkfun-Artemis:XCVR_CGGBP.35.6.A.02, symbol CGGBP.35.6.A.02:CGGBP.35.6.A.02
- added R6: R, Resistor_SMD:R_0805_2012Metric_Pad1.15x1.40mm_HandSolder, symbol Device:R
- added U5: SGGP.12.4.A.02, RF_Antenna:SGGP.12.4.A.02, symbol Sparkfun~Artemis:SGGP.12.4.A.02
- renumbered C10 to C11, U3 to U4
Connections:
- wire segments 20 -> 35
Changed lines of the file:
@@
 $EndDescr
 $Comp
-L RF_GPS:MAX-8Q U3
+L RF_GPS:MAX-8Q U4
 U 1 1 5E6E6DC2
 P 5750 3450
-F 0 "U3" H 5750 2661 50  0000 C CNN
+F 0 "U4" H 5750 2661 50  0000 C CNN
 F 1 "MAX-8Q" H 5750 2570 50  0000 C CNN
 F 2 "RF_GPS:ublox_MAX" H 6150 2800 50  0001 C CNN
@@
 $EndComp
 $Comp
-L power:GND #PWR0119
+L power:GND #PWR022
 U 1 1 5E6E7D04
 P 4400 4400
-F 0 "#PWR0119" H 4400 4150 50  0001 C CNN
+F 0 "#PWR022" H 4400 4150 50  0001 C CNN
 F 1 "GND" H 4405 4227 50  0000 C CNN
 F 2 "" H 4400 4400 50  0001 C CNN
@@
 $EndComp
 $Comp
-L power:+3.3V #PWR0120
+L power:+3.3V #PWR021
 U 1 1 5E6E8495
 P 4400 2500
-F 0 "#PWR0120" H 4400 2350 50  0001 C CNN
+F 0 "#PWR021" H 4400 2350 50  0001 C CNN
 F 1 "+3.3V" H 4415 2673 50  0000 C CNN
 F 2 "" H 4400 2500 50  0001 C CNN
@@
 	6350 3450 6700 3450
 $Comp
-L pspice:CAP C10
+L pspice:CAP C11
 U 1 1 5E6EAF56
 P 4400 3550
-F 0 "C10" H 4578 3596 50  0000 L CNN
+F 0 "C11" H 4578 3596 50  0000 L CNN
 F 1 "0.1uF" H 4578 3505 50  0000 L CNN
 F 2 "Capacitor_SMD:C_0805_2012Metric_Pad1.15x1.40mm_HandSolder" H 4400 3550 50  0001 C CNN
@@
 Text HLabel 4600 3050 0    50   Input ~ 0
 RX
-$Comp
-L CGGBP.35.6.A.02:CGGBP.35.6.A.02 AE1
-U 1 1 5E756F28
-P 6900 3100
-F 0 "AE1" H 7168 3135 50  0000 L CNN
-F 1 "CGGBP.35.6.A.02" H 7168 3044 50  0000 L CNN
-F 2 "Sparkfun-Artemis:XCVR_CGGBP.35.6.A.02" H 6900 3100 50  0001 L BNN
-F 3 "Taoglas" H 6900 3100 50  0001 L BNN
-	1    6900 3100
-	1    0    0    -1
-$EndComp
 $Comp
 L Device:Ferrite_Bead_Small FB1
@@
 Wire Wire Line
 	5100 3050 5150 3050
-Wire Wire Line
-	6700 3450 6700 3300
-Wire Wire Line
-	6700 3300 6800 3300
-$Comp
-L power:GND #PWR0122
-U 1 1 5E7583F9
-P 6600 3200
-F 0 "#PWR0122" H 6600 2950 50  0001 C CNN
-F 1 "GND" H 6605 3027 50  0000 C CNN
-F 2 "" H 6600 3200 50  0001 C CNN
-F 3 "" H 6600 3200 50  0001 C CNN
-	1    6600 3200
-	1    0    0    -1
-$EndComp
-Wire Wire Line
-	6600 3200 6600 3100
-Wire Wire Line
-	6600 3100 6800 3100
+$Comp
+L Device:R R6
+U 1 1 5E765CE3
+P 6850 3450
+F 0 "R6" V 6643 3450 50  0000 C CNN
+F 1 "R" V 6734 3450 50  0000 C CNN
+F 2 "Resistor_SMD:R_0805_2012Metric_Pad1.15x1.40mm_HandSolder" V 6780 3450 50  0001 C CNN
+F 3 "~" H 6850 3450 50  0001 C CNN
+	1    6850 3450
+	0    1    1    0
+$EndComp
+$Comp
+L Sparkfun~Artemis:SGGP.12.4.A.02 U5
+U 1 1 5E7667EA
+P 7100 2700
+F 0 "U5" H 7100 2700 50  0001 L BNN
+F 1 "SGGP.12.4.A.02" H 7100 2700 50  0001 L BNN
+F 2 "RF_Antenna:SGGP.12.4.A.02" H 7100 2700 50  0001 L BNN
+F 3 "" H 7100 2700 50  0001 C CNN
+	1    7100 2700
+	1    0    0    -1
+$EndComp
+Wire Wire Line
+	7000 3450 8250 3450
+Wire Wire Line
+	8250 2800 8000 2800
+$Comp
+L power:GND #PWR023
+U 1 1 5E767B82
+P 7000 2950
+F 0 "#PWR023" H 7000 2700 50  0001 C CNN
+F 1 "GND" H 7005 2777 50  0000 C CNN
+F 2 "" H 7000 2950 50  0001 C CNN
+F 3 "" H 7000 2950 50  0001 C CNN
+	1    7000 2950
+	1    0    0    -1
+$EndComp
+Wire Wire Line
+	8250 2800 8250 3450
+Wire Wire Line
+	7100 2500 7000 2500
+Wire Wire Line
+	7000 2500 7000 2600
+Wire Wire Line
+	7100 2800 7000 2800
+Connection ~ 7000 2800
+Wire Wire Line
+	7000 2800 7000 2950
+Wire Wire Line
+	7100 2700 7000 2700
+Connection ~ 7000 2700
+Wire Wire Line
+	7000 2700 7000 2800
+Wire Wire Line
+	7100 2600 7000 2600
+Connection ~ 7000 2600
+Wire Wire Line
+	7000 2600 7000 2700
+$Comp
+L power:GND #PWR024
+U 1 1 5E76ED42
+P 8100 2950
+F 0 "#PWR024" H 8100 2700 50  0001 C CNN
+F 1 "GND" H 8105 2777 50  0000 C CNN
+F 2 "" H 8100 2950 50  0001 C CNN
+F 3 "" H 8100 2950 50  0001 C CNN
+	1    8100 2950
+	1    0    0    -1
+$EndComp
+Wire Wire Line
+	8000 2500 8100 2500
+Wire Wire Line
+	8100 2500 8100 2600
+Wire Wire Line
+	8000 2600 8100 2600
+Connection ~ 8100 2600
+Wire Wire Line
+	8100 2600 8100 2700
+Wire Wire Line
+	8000 2700 8100 2700
+Wire Wire Line
+	8000 2900 8100 2900
+Wire Wire Line
+	8100 2900 8100 2950
+$Comp
+L power:GND #PWR025
+U 1 1 5E765E1B
+P 8300 2600
+F 0 "#PWR025" H 8300 2350 50  0001 C CNN
+F 1 "GND" V 8305 2472 50  0000 R CNN
+F 2 "" H 8300 2600 50  0001 C CNN
+F 3 "" H 8300 2600 50  0001 C CNN
+	1    8300 2600
+	0    -1   -1   0
+$EndComp
+Wire Wire Line
+	8100 2600 8300 2600
 $EndSCHEMATC

Commit message: schamatics finalized
Parts:
- added C19, C2: CAP, Capacitor_SMD:C_0805_2012Metric_Pad1.15x1.40mm_HandSolder, symbol pspice:CAP
- added D4: LED, LED_SMD:LED_0805_2012Metric_Pad1.15x1.40mm_HandSolder, symbol Device:LED
- added FL1: SAFFA1G58KA0F0A, Filter:Filter_1411-5_1.4x1.1mm, symbol Filter:SAFFA1G58KA0F0A
- added L1: INDUCTOR, Inductor_SMD:L_0805_2012Metric_Pad1.15x1.40mm_HandSolder, symbol pspice:INDUCTOR
- added U9: MAX2686, Package_BGA:WLP-4_0.86x0.86mm_P0.4mm, symbol Sparkfun~Artemis:MAX2686
Connections:
- net labels added: RESET
- wire segments 35 -> 52
- no-connect marks 0 -> 6
Other:
- moved on the sheet: C11, FB1, FB2, U4

Commit message: updates to routing and fix commit
Parts:
- C19: value CAP -> 100 nf
- C2: value CAP -> 10 pf
- D4: Man (none) -> Kingbright; Man part # (none) -> APTD2012LSURCK; Mouser (none) -> 604-APTD2012LSURCK
- L1: value INDUCTOR -> 6.8 nH
- R6: value R -> 750
- U5: symbol Sparkfun~Artemis:SGGP.12.4.A.02 -> Mini_GPS_Tracker-rescue:SGGP.12.4.A.02-Sparkfun_Artemis-Mini_GPS_Tracker-rescue
- U9: symbol Sparkfun~Artemis:MAX2686 -> Mini_GPS_Tracker-rescue:MAX2686-Sparkfun_Artemis-Mini_GPS_Tracker-rescue
Changed lines of the file:
@@
 	3700 3900 3750 3900
 $Comp
-L Sparkfun~Artemis:SGGP.12.4.A.02 U5
+L Mini_GPS_Tracker-rescue:SGGP.12.4.A.02-Sparkfun_Artemis-Mini_GPS_Tracker-rescue U5
 U 1 1 5E7667EA
 P 7850 1850
@@
 P 5150 4850
 F 0 "R6" H 5220 4896 50  0000 L CNN
-F 1 "R" H 5220 4805 50  0000 L CNN
+F 1 "750" H 5220 4805 50  0000 L CNN
 F 2 "Resistor_SMD:R_0805_2012Metric_Pad1.15x1.40mm_HandSolder" V 5080 4850 50  0001 C CNN
 F 3 "~" H 5150 4850 50  0001 C CNN
@@
 F 1 "LED" V 5098 5083 50  0000 R CNN
 F 2 "LED_SMD:LED_0805_2012Metric_Pad1.15x1.40mm_HandSolder" H 5150 5200 50  0001 C CNN
-F 3 "~" H 5150 5200 50  0001 C CNN
+F 3 "https://www.mouser.com/datasheet/2/216/APTD2012LSURCK-1101937.pdf" H 5150 5200 50  0001 C CNN
+F 4 "APTD2012LSURCK " V 5150 5200 50  0001 C CNN "Man part #"
+F 5 "Kingbright " V 5150 5200 50  0001 C CNN "Man"
+F 6 "604-APTD2012LSURCK " V 5150 5200 50  0001 C CNN "Mouser"
 	1    5150 5200
 	0    -1   -1   0
@@
 $EndComp
 $Comp
-L Sparkfun~Artemis:MAX2686 U9
+L Mini_GPS_Tracker-rescue:MAX2686-Sparkfun_Artemis-Mini_GPS_Tracker-rescue U9
 U 1 1 5E78E34D
 P 7850 4600
@@
 P 8700 4300
 F 0 "L1" H 8700 4515 50  0000 C CNN
-F 1 "INDUCTOR" H 8700 4424 50  0000 C CNN
+F 1 "6.8 nH" H 8700 4424 50  0000 C CNN
 F 2 "Inductor_SMD:L_0805_2012Metric_Pad1.15x1.40mm_HandSolder" H 8700 4300 50  0001 C CNN
 F 3 "~" H 8700 4300 50  0001 C CNN
@@
 P 8350 3650
 F 0 "C2" H 8528 3696 50  0000 L CNN
-F 1 "CAP" H 8528 3605 50  0000 L CNN
+F 1 "10 pf" H 8528 3605 50  0000 L CNN
 F 2 "Capacitor_SMD:C_0805_2012Metric_Pad1.15x1.40mm_HandSolder" H 8350 3650 50  0001 C CNN
 F 3 "~" H 8350 3650 50  0001 C CNN
@@
 P 9250 4300
 F 0 "C19" V 8935 4300 50  0000 C CNN
-F 1 "CAP" V 9026 4300 50  0000 C CNN
+F 1 "100 nf" V 9026 4300 50  0000 C CNN
 F 2 "Capacitor_SMD:C_0805_2012Metric_Pad1.15x1.40mm_HandSolder" H 9250 4300 50  0001 C CNN
 F 3 "~" H 9250 4300 50  0001 C CNN
@@
 Wire Wire Line
 	8750 1950 9550 1950
+Connection ~ 9500 4300
+Wire Wire Line
+	9500 4300 9550 4300
+Wire Wire Line
+	8950 4300 9000 4300
 Wire Wire Line
 	8350 4300 8450 4300
-Connection ~ 9500 4300
-Wire Wire Line
-	9500 4300 9550 4300
-Wire Wire Line
-	8950 4300 9000 4300
 $EndSCHEMATC
