File: Mini_GPS_Tracker/Storage.sch (KiCad schematic (older format))
At the start: 1 part, among them U8 W25Q128JVS

Commit message: Adding BNO055 Motion co-processor
Parts:
- U8: symbol Memory_Flash:W25Q128JVS -> Mini_GPS_Tracker-rescue:W25Q128JVS-Memory_Flash
Changed lines of the file:
@@
 EESchema Schematic File Version 4
+LIBS:Mini_GPS_Tracker-cache
 EELAYER 30 0
 EELAYER END
 $Descr A4 11693 8268
 encoding utf-8
-Sheet 6 6
+Sheet 6 7
 Title ""
 Date ""
@@
 $EndDescr
 $Comp
-L Memory_Flash:W25Q128JVS U8
+L Mini_GPS_Tracker-rescue:W25Q128JVS-Memory_Flash U8
 U 1 1 5E7A9464
 P 5700 3900
