File: Mini_GPS_Tracker/Storage.sch (KiCad schematic (older format))
At the start: 1 part, among them U8 W25Q128JVS

Commit message: updates to routing and fix commit
Parts:
- U8: symbol Memory_Flash:W25Q128JVS -> Mini_GPS_Tracker-rescue:W25Q128JVS-Memory_Flash-Mini_GPS_Tracker-rescue
Changed lines of the file:
@@
 $EndDescr
 $Comp
-L Memory_Flash:W25Q128JVS U8
+L Mini_GPS_Tracker-rescue:W25Q128JVS-Memory_Flash-Mini_GPS_Tracker-rescue U8
 U 1 1 5E7A9464
 P 5700 3900
+AR Path="/5E7A9464" Ref="U8"  Part="1"
+AR Path="/5E7CBED1/5E7A9464" Ref="U8"  Part="1"
 F 0 "U8" H 5700 4481 50  0000 C CNN
 F 1 "W25Q128JVS" H 5700 4390 50  0000 C CNN

Commit message: Add files via upload
Updates schematics
Changed lines of the file:
@@
 EESchema Schematic File Version 4
+LIBS:Mini_GPS_Tracker-cache
 EELAYER 30 0
 EELAYER END
 $Descr A4 11693 8268
 encoding utf-8
-Sheet 6 6
+Sheet 6 10
 Title ""
 Date ""
@@
 Wire Wire Line
 	6200 3700 6400 3700
+Connection ~ 5200 3800
 $EndSCHEMATC
