File: Mini_GPS_Tracker/Transmitter.sch (KiCad schematic (older format))
At the start: 4 parts, among them J3 901-10512-1, U6 XBee_SMT

Commit message: added bluetooth wifi module
Parts:
- added TP? (x5): TestPoint, symbol Connector:TestPoint
- added U?: LBEE5KL1DX-TEMP, XCVR_LBEE5KL1DX-TEMP, symbol Sparkfun~Artemis:LBEE5KL1DX-TEMP
Connections:
- net labels added: murata_cts, murata_rts, murata_rx, murata_tx
- wire segments 22 -> 33
- no-connect marks 20 -> 25
Other:
- moved on the sheet: C12, C13, J3, U6

Commit message: added stm core connections
Parts:
- U10: renamed from U?; footprint XCVR_LBEE5KL1DX-TEMP -> Sparkfun-Artemis:XCVR_LBEE5KL1DX-TEMP
- gave numbers to parts that had none: 5
Changed lines of the file:
@@
 	3750 1100 3750 1300
 $Comp
-L Sparkfun~Artemis:LBEE5KL1DX-TEMP U?
+L Sparkfun~Artemis:LBEE5KL1DX-TEMP U10
 U 1 1 5E8A8D4C
 P 8250 3700
-F 0 "U?" H 8250 5167 50  0000 C CNN
+F 0 "U10" H 8250 5167 50  0000 C CNN
 F 1 "LBEE5KL1DX-TEMP" H 8250 5076 50  0000 C CNN
-F 2 "XCVR_LBEE5KL1DX-TEMP" H 8250 3700 50  0001 L BNN
+F 2 "Sparkfun-Artemis:XCVR_LBEE5KL1DX-TEMP" H 8250 3700 50  0001 L BNN
 F 3 "12.26 USD" H 8250 3700 50  0001 L BNN
 F 4 "LBEE5KL1DX-TEMP" H 8250 3700 50  0001 L BNN "Field4"
@@
 NoConn ~ 6950 3800
 $Comp
-L power:GND #PWR?
+L power:GND #PWR0129
 U 1 1 5E8ABDFC
 P 9700 4900
-F 0 "#PWR?" H 9700 4650 50  0001 C CNN
+F 0 "#PWR0129" H 9700 4650 50  0001 C CNN
 F 1 "GND" H 9705 4727 50  0000 C CNN
 F 2 "" H 9700 4900 50  0001 C CNN
@@
 	9700 4800 9700 4900
 $Comp
-L Connector:TestPoint TP?
+L Connector:TestPoint TP4
 U 1 1 5E8ACFDF
 P 6750 3600
-F 0 "TP?" V 6945 3672 50  0000 C CNN
+F 0 "TP4" V 6945 3672 50  0000 C CNN
 F 1 "TestPoint" V 6854 3672 50  0000 C CNN
 F 2 "" H 6950 3600 50  0001 C CNN
@@
 $EndComp
 $Comp
-L Connector:TestPoint TP?
+L Connector:TestPoint TP3
 U 1 1 5E8AEBF2
 P 6750 3100
-F 0 "TP?" V 6945 3172 50  0000 C CNN
+F 0 "TP3" V 6945 3172 50  0000 C CNN
 F 1 "TestPoint" V 6854 3172 50  0000 C CNN
 F 2 "" H 6950 3100 50  0001 C CNN
@@
 $EndComp
 $Comp
-L Connector:TestPoint TP?
+L Connector:TestPoint TP5
 U 1 1 5E8AFDE5
 P 9650 3100
-F 0 "TP?" V 9604 3288 50  0000 L CNN
+F 0 "TP5" V 9604 3288 50  0000 L CNN
 F 1 "TestPoint" V 9695 3288 50  0000 L CNN
 F 2 "" H 9850 3100 50  0001 C CNN
@@
 $EndComp
 $Comp
-L Connector:TestPoint TP?
+L Connector:TestPoint TP2
 U 1 1 5E8B43E2
 P 6250 3500
-F 0 "TP?" V 6445 3572 50  0000 C CNN
+F 0 "TP2" V 6445 3572 50  0000 C CNN
 F 1 "TestPoint" V 6354 3572 50  0000 C CNN
 F 2 "" H 6450 3500 50  0001 C CNN
@@
 $EndComp
 $Comp
-L Connector:TestPoint TP?
+L Connector:TestPoint TP1
 U 1 1 5E8B53B7
 P 5800 3400
-F 0 "TP?" V 5995 3472 50  0000 C CNN
+F 0 "TP1" V 5995 3472 50  0000 C CNN
 F 1 "TestPoint" V 5904 3472 50  0000 C CNN
 F 2 "" H 6000 3400 50  0001 C CNN
