File: Mini_GPS_Tracker/Power.sch (KiCad schematic (older format))
At the start: 5 parts, among them J3 XT60-M, U4 LD1117S33TR_SOT223

Commit message: updated antenna;
Parts:
- removed J3: XT60-M, Sparkfun-Artemis:AMASS_XT60-M, symbol XT60-M:XT60-M
- added J2: Screw_Terminal_01x02, Connector_AMASS:AMASS_XT30UPB-F_1x02_P5.0mm_Vertical, symbol Connector:Screw_Terminal_01x02
- renumbered C12 to C10, C11 to C9, U4 to U3
Other:
- moved on the sheet: D3
Changed lines of the file:
@@
 $Descr A4 11693 8268
 encoding utf-8
-Sheet 3 5
+Sheet 1 5
 Title ""
 Date ""
@@
 $EndDescr
 $Comp
-L Regulator_Linear:LD1117S33TR_SOT223 U4
+L Regulator_Linear:LD1117S33TR_SOT223 U3
 U 1 1 5E6E6EA8
 P 5250 4250
-F 0 "U4" H 5250 4492 50  0000 C CNN
+F 0 "U3" H 5250 4492 50  0000 C CNN
 F 1 "LD1117S33TR_SOT223" H 5250 4401 50  0000 C CNN
 F 2 "Package_TO_SOT_SMD:SOT-223-3_TabPin2" H 5250 4450 50  0001 C CNN
@@
 $EndComp
 $Comp
-L power:GND #PWR0121
+L power:GND #PWR019
 U 1 1 5E6E846B
 P 5250 5000
-F 0 "#PWR0121" H 5250 4750 50  0001 C CNN
+F 0 "#PWR019" H 5250 4750 50  0001 C CNN
 F 1 "GND" H 5255 4827 50  0000 C CNN
 F 2 "" H 5250 5000 50  0001 C CNN
@@
 $EndComp
 $Comp
-L pspice:CAP C11
+L pspice:CAP C9
 U 1 1 5E6EAADE
 P 4550 4600
-F 0 "C11" H 4728 4646 50  0000 L CNN
+F 0 "C9" H 4728 4646 50  0000 L CNN
 F 1 "100nF" H 4728 4555 50  0000 L CNN
 F 2 "Capacitor_SMD:C_0805_2012Metric_Pad1.15x1.40mm_HandSolder" H 4550 4600 50  0001 C CNN
@@
 $EndComp
 $Comp
-L pspice:CAP C12
+L pspice:CAP C10
 U 1 1 5E6EB3FA
 P 6050 4600
-F 0 "C12" H 6228 4646 50  0000 L CNN
+F 0 "C10" H 6228 4646 50  0000 L CNN
 F 1 "100nF" H 6228 4555 50  0000 L CNN
 F 2 "Capacitor_SMD:C_0805_2012Metric_Pad1.15x1.40mm_HandSolder" H 6050 4600 50  0001 C CNN
@@
 $EndComp
 $Comp
-L power:+3.3V #PWR0123
+L power:+3.3V #PWR020
 U 1 1 5E6E8A06
 P 6050 2750
-F 0 "#PWR0123" H 6050 2600 50  0001 C CNN
+F 0 "#PWR020" H 6050 2600 50  0001 C CNN
 F 1 "+3.3V" H 6065 2923 50  0000 C CNN
 F 2 "" H 6050 2750 50  0001 C CNN
@@
 Wire Wire Line
 	4950 4250 4550 4250
-Connection ~ 4550 4250
 Wire Wire Line
 	4550 4250 4550 4350
@@
 L pspice:DIODE D3
 U 1 1 5E7589B4
-P 6050 3750
-F 0 "D3" V 6096 3622 50  0000 R CNN
-F 1 "DIODE" V 6005 3622 50  0000 R CNN
-F 2 "Diode_SMD:D_0805_2012Metric_Pad1.15x1.40mm_HandSolder" H 6050 3750 50  0001 C CNN
-F 3 "~" H 6050 3750 50  0001 C CNN
-	1    6050 3750
+P 4550 3600
+F 0 "D3" V 4596 3472 50  0000 R CNN
+F 1 "DIODE" V 4505 3472 50  0000 R CNN
+F 2 "Diode_SMD:D_0805_2012Metric_Pad1.15x1.40mm_HandSolder" H 4550 3600 50  0001 C CNN
+F 3 "~" H 4550 3600 50  0001 C CNN
+	1    4550 3600
+	0    1    1    0
+$EndComp
+Connection ~ 6050 4250
+$Comp
+L power:GND #PWR018
+U 1 1 5E75AA69
+P 4450 3100
+F 0 "#PWR018" H 4450 2850 50  0001 C CNN
+F 1 "GND" H 4455 2927 50  0000 C CNN
+F 2 "" H 4450 3100 50  0001 C CNN
+F 3 "" H 4450 3100 50  0001 C CNN
+	1    4450 3100
+	1    0    0    -1
+$EndComp
+Wire Wire Line
+	4450 3100 4450 2900
+$Comp
+L Connector:Screw_Terminal_01x02 J2
+U 1 1 5E7654CA
+P 4450 2700
+F 0 "J2" V 4414 2512 50  0000 R CNN
+F 1 "Screw_Terminal_01x02" V 4323 2512 50  0000 R CNN
+F 2 "Connector_AMASS:AMASS_XT30UPB-F_1x02_P5.0mm_Vertical" H 4450 2700 50  0001 C CNN
+F 3 "~" H 4450 2700 50  0001 C CNN
+	1    4450 2700
 	0    -1   -1   0
 $EndComp
 Wire Wire Line
-	6050 2750 6050 3550
+	6050 2750 6050 4250
 Wire Wire Line
-	6050 4250 6050 3950
-Connection ~ 6050 4250
-$Comp
-L XT60-M:XT60-M J3
-U 1 1 5E759DF8
-P 4450 2850
-F 0 "J3" V 4389 2620 50  0000 R CNN
-F 1 "XT60-M" V 4298 2620 50  0000 R CNN
-F 2 "Sparkfun-Artemis:AMASS_XT60-M" H 4450 2850 50  0001 L BNN
-F 3 "1.2" H 4450 2850 50  0001 L BNN
-F 4 "IPC-7251" H 4450 2850 50  0001 L BNN "Field4"
-F 5 "AMASS" H 4450 2850 50  0001 L BNN "Field5"
-	1    4450 2850
-	0    -1   -1   0
-$EndComp
-$Comp
-L power:GND #PWR02
-U 1 1 5E75AA69
-P 4350 3350
-F 0 "#PWR02" H 4350 3100 50  0001 C CNN
-F 1 "GND" H 4355 3177 50  0000 C CNN
-F 2 "" H 4350 3350 50  0001 C CNN
-F 3 "" H 4350 3350 50  0001 C CNN
-	1    4350 3350
-	1    0    0    -1
-$EndComp
+	4550 2900 4550 3400
 Wire Wire Line
-	4550 3150 4550 4250
-Wire Wire Line
-	4350 3350 4350 3150
+	4550 3800 4550 4250
+Connection ~ 4550 4250
 $EndSCHEMATC

Commit message: schamatics finalized
Parts:
- added R1: 10k, Resistor_SMD:R_0805_2012Metric_Pad1.15x1.40mm_HandSolder, symbol Device:R
- added R3: 3k, Resistor_SMD:R_0805_2012Metric_Pad1.15x1.40mm_HandSolder, symbol Device:R
- added SW2: MLL1200S, Sparkfun-Artemis:SW_MLL1200S, symbol Sparkfun~Artemis:MLL1200S
- C10: value 100nF -> 10uF
Connections:
- net labels added: V_Bat_Measure
- wire segments 13 -> 24
Other:
- moved on the sheet: C10, C9, D3, J2, U3

Commit message: updates to routing and fix commit
Parts:
- SW2: symbol Sparkfun~Artemis:MLL1200S -> Mini_GPS_Tracker-rescue:MLL1200S-Sparkfun_Artemis-Mini_GPS_Tracker-rescue
Connections:
- wire segments 24 -> 27
- no-connect marks 0 -> 1
Changed lines of the file:
@@
 Wire Wire Line
 	5250 1900 5250 2000
-Wire Wire Line
-	6750 2450 6750 2950
 $Comp
 L Connector:Screw_Terminal_01x02 J2
@@
 	4050 3950 4050 4000
 $Comp
-L power:PWR_FLAG #FLG0101
-U 1 1 5E78C7E9
-P 6750 2950
-F 0 "#FLG0101" H 6750 3025 50  0001 C CNN
-F 1 "PWR_FLAG" V 6750 3078 50  0000 L CNN
-F 2 "" H 6750 2950 50  0001 C CNN
-F 3 "~" H 6750 2950 50  0001 C CNN
-	1    6750 2950
-	0    1    1    0
-$EndComp
-Connection ~ 6750 2950
-Wire Wire Line
-	6750 2950 6750 3950
-$Comp
 L power:PWR_FLAG #FLG0102
 U 1 1 5E78D09D
@@
 	0    1    1    0
 $EndComp
-Connection ~ 5250 2000
 $Comp
 L power:PWR_FLAG #FLG0103
@@
 	5150 2000 5150 1900
 $Comp
-L Sparkfun~Artemis:MLL1200S SW2
+L Mini_GPS_Tracker-rescue:MLL1200S-Sparkfun_Artemis-Mini_GPS_Tracker-rescue SW2
 U 1 1 5E7E93B5
 P 5650 2800
@@
 $EndComp
 Wire Wire Line
-	5250 2000 5250 2600
-Wire Wire Line
 	5250 2800 5250 3100
 $Comp
@@
 Wire Wire Line
 	6050 2900 6050 3050
+Wire Wire Line
+	5250 2000 5250 2150
+Wire Wire Line
+	5250 2150 6050 2150
+Wire Wire Line
+	6050 2150 6050 2700
+Connection ~ 5250 2000
+NoConn ~ 5250 2600
+Wire Wire Line
+	6750 2450 6750 3950
+$Comp
+L power:PWR_FLAG #FLG0101
+U 1 1 5E83E3CB
+P 5650 3450
+F 0 "#FLG0101" H 5650 3525 50  0001 C CNN
+F 1 "PWR_FLAG" H 5650 3623 50  0000 C CNN
+F 2 "" H 5650 3450 50  0001 C CNN
+F 3 "~" H 5650 3450 50  0001 C CNN
+	1    5650 3450
+	1    0    0    -1
+$EndComp
+Wire Wire Line
+	5250 3600 5650 3600
+Wire Wire Line
+	5650 3600 5650 3450
 $EndSCHEMATC
