File: Mini_GPS_Tracker/Power.sch (KiCad schematic (older format))
At the start: 8 parts, among them J2 Screw_Terminal_01x02, SW2 MLL1200S, U3 LD1117S33TR_SOT223

Commit message: Add files via upload
Adding 100 pin MCU
Connections:
- net VBUS: now reaches D3.1 (K), SW2.3
Changed lines of the file:
@@
 EESchema Schematic File Version 4
-LIBS:Mini_GPS_Tracker-cache
 EELAYER 30 0
 EELAYER END
 $Descr A4 11693 8268
 encoding utf-8
-Sheet 3 10
+Sheet 3 11
 Title ""
 Date ""
@@
 	0    -1   -1   0
 $EndComp
-Wire Wire Line
-	5150 2100 5150 2000
-$Comp
-L power:GND #PWR018
-U 1 1 5E75AA69
-P 5150 2100
-F 0 "#PWR018" H 5150 1850 50  0001 C CNN
-F 1 "GND" H 5155 1927 50  0000 C CNN
-F 2 "" H 5150 2100 50  0001 C CNN
-F 3 "" H 5150 2100 50  0001 C CNN
-	1    5150 2100
-	1    0    0    -1
-$EndComp
 Connection ~ 6750 3950
 $Comp
@@
 $EndComp
 Wire Wire Line
-	5250 2800 5250 3100
+	5250 2800 5250 3000
 $Comp
 L power:GND #PWR0115
@@
 Wire Wire Line
 	5650 3600 5650 3450
+Text HLabel 3900 3000 0    50   Input ~ 0
+VBUS
+Connection ~ 5250 3000
+Wire Wire Line
+	5250 3000 5250 3100
+Wire Wire Line
+	3900 3000 5250 3000
+Wire Wire Line
+	5150 2100 5150 2000
+$Comp
+L power:GND #PWR018
+U 1 1 5E75AA69
+P 5150 2100
+F 0 "#PWR018" H 5150 1850 50  0001 C CNN
+F 1 "GND" H 5155 1927 50  0000 C CNN
+F 2 "" H 5150 2100 50  0001 C CNN
+F 3 "" H 5150 2100 50  0001 C CNN
+	1    5150 2100
+	1    0    0    -1
+$EndComp
 $EndSCHEMATC
