File: Mini_GPS_Tracker/Mini_GPS_Tracker.sch (KiCad schematic (older format))
At the start: 24 parts, among them J1 USB_C_Receptacle, J4 Conn_ARM_JTAG_SWD_10, SW1 SW_Push, U1 FT230XS, Y1 32.786 KHz

Commit message: added stm chip
Parts:
- removed C20: 100 nf, Capacitor_SMD:C_0805_2012Metric, symbol Device:C
- removed C3: 0.1uF, Capacitor_SMD:C_0805_2012Metric_Pad1.15x1.40mm_HandSolder, symbol pspice:CAP
- removed C5: 10nF, Capacitor_SMD:C_0805_2012Metric_Pad1.15x1.40mm_HandSolder, symbol pspice:CAP
- removed D1, D2: LED, LED_SMD:LED_0805_2012Metric_Pad1.15x1.40mm_HandSolder, symbol Device:LED
- removed MD1: SPARKFUN_WRL-15376, Sparkfun-Artemis:SPARKFUN_WRL-15376, symbol Mini_GPS_Tracker-rescue:SPARKFUN_WRL-15376-Sparkfun_Artemis-Mini_GPS_Tracker-re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
- removed R4, R5: 1K, Resistor_SMD:R_0805_2012Metric_Pad1.15x1.40mm_HandSolder, symbol Device:R
- removed U1: FT230XS, Package_SO:SSOP-16_3.9x4.9mm_P0.635mm, symbol Interface_USB:FT230XS
- added U10: STMICROELECTRONICS_STM32H747XIH6, Package_BGA:TFBGA-265_14x14mm_Layout17x17_P0.8mm, symbol STM32H747XIH6:STMICROELECTRONICS_STM32H747XIH6
Connections:
- wire segments 128 -> 72
- no-connect marks 48 -> 15
Other:
- moved on the sheet: C6, C7, Y1

Commit message: added bluetooth wifi module
Parts:
- removed U10: STMICROELECTRONICS_STM32H747XIH6, Package_BGA:TFBGA-265_14x14mm_Layout17x17_P0.8mm, symbol STM32H747XIH6:STMICROELECTRONICS_STM32H747XIH6
- added IC?: STM32H747XIH6, BGA265C80P17X17_1400X1400X110, symbol Sparkfun~Artemis:STM32H747XIH6
Connections:
- wire segments 72 -> 89
Changed lines of the file:
@@
-	1    0    0    -1
-$EndComp
-$Comp
-L STM32H747XIH6:STMICROELECTRONICS_STM32H747XIH6 U10
-U 1 1 5E872F9C
-P -4900 -4850
-F 0 "U10" H -4200 -4975 50  0000 C CNN
-F 1 "STMICROELECTRONICS_STM32H747XIH6" H -4900 -4850 50  0001 L BNN
-F 2 "Package_BGA:TFBGA-265_14x14mm_Layout17x17_P0.8mm" H -4900 -4850 50  0001 C CNN
-F 3 "" H -4900 -4850 50  0001 C CNN
-	1    -4900 -4850
-	1    0    0    -1
-$EndComp
-$Comp
-L STM32H747XIH6:STMICROELECTRONICS_STM32H747XIH6 U10
-U 2 1 5E89920D
-P -2550 -4000
-F 0 "U10" H -1650 -4124 50  0000 C CNN
-F 1 "STMICROELECTRONICS_STM32H747XIH6" H -2550 -4000 50  0001 L BNN
-F 2 "Package_BGA:TFBGA-265_14x14mm_Layout17x17_P0.8mm" H -2550 -4000 50  0001 C CNN
-F 3 "" H -2550 -4000 50  0001 C CNN
-	2    -2550 -4000
-	1    0    0    -1
-$EndComp
-$Comp
-L STM32H747XIH6:STMICROELECTRONICS_STM32H747XIH6 U10
-U 3 1 5E8A86B1
-P 300 -4800
-F 0 "U10" H 1150 -4925 50  0000 C CNN
-F 1 "STMICROELECTRONICS_STM32H747XIH6" H 300 -4800 50  0001 L BNN
-F 2 "Package_BGA:TFBGA-265_14x14mm_Layout17x17_P0.8mm" H 300 -4800 50  0001 C CNN
-F 3 "" H 300 -4800 50  0001 C CNN
-	3    300  -4800
-	1    0    0    -1
-$EndComp
-$Comp
-L STM32H747XIH6:STMICROELECTRONICS_STM32H747XIH6 U10
-U 4 1 5E8C3A7F
-P 3500 -4650
-F 0 "U10" H 4250 -4775 50  0000 C CNN
-F 1 "STMICROELECTRONICS_STM32H747XIH6" H 3500 -4650 50  0001 L BNN
-F 2 "Package_BGA:TFBGA-265_14x14mm_Layout17x17_P0.8mm" H 3500 -4650 50  0001 C CNN
-F 3 "" H 3500 -4650 50  0001 C CNN
-	4    3500 -4650
-	1    0    0    -1
-$EndComp
-$Comp
-L STM32H747XIH6:STMICROELECTRONICS_STM32H747XIH6 U10
-U 5 1 5E8E416C
-P 6250 -4500
-F 0 "U10" H 6950 -4625 50  0000 C CNN
-F 1 "STMICROELECTRONICS_STM32H747XIH6" H 6250 -4500 50  0001 L BNN
-F 2 "Package_BGA:TFBGA-265_14x14mm_Layout17x17_P0.8mm" H 6250 -4500 50  0001 C CNN
-F 3 "" H 6250 -4500 50  0001 C CNN
-	5    6250 -4500
 	1    0    0    -1
 $EndComp
@@
 	1    0    0    -1
 $EndComp
+$Comp
+L Sparkfun~Artemis:STM32H747XIH6 IC?
+U 1 1 5E894707
+P 14100 -2900
+F 0 "IC?" H 15100 -2635 50  0000 C CNN
+F 1 "STM32H747XIH6" H 15100 -2726 50  0000 C CNN
+F 2 "BGA265C80P17X17_1400X1400X110" H 15950 -2800 50  0001 L CNN
+F 3 "https://www.st.com/en/microcontrollers-microprocessors/stm32h747xi.html" H 15950 -2900 50  0001 L CNN
+F 4 "ARM Microcontrollers - MCU" H 15950 -3000 50  0001 L CNN "Description"
+F 5 "1.1" H 15950 -3100 50  0001 L CNN "Height"
+F 6 "STMicroelectronics" H 15950 -3200 50  0001 L CNN "Manufacturer_Name"
+F 7 "STM32H747XIH6" H 15950 -3300 50  0001 L CNN "Manufacturer_Part_Number"
+F 8 "511-STM32H747XIH6" H 15950 -3400 50  0001 L CNN "Mouser Part Number"
+F 9 "https://www.mouser.com/Search/Refine.aspx?Keyword=511-STM32H747XIH6" H 15950 -3500 50  0001 L CNN "Mouser Price/Stock"
+F 10 "" H 15950 -3600 50  0001 L CNN "RS Part Number"
+F 11 "" H 15950 -3700 50  0001 L CNN "RS Price/Stock"
+	1    14100 -2900
+	1    0    0    -1
+$EndComp
+$Comp
+L power:+3.3V #PWR?
+U 1 1 5E8BD97D
+P 13900 10500
+F 0 "#PWR?" H 13900 10350 50  0001 C CNN
+F 1 "+3.3V" H 13915 10673 50  0000 C CNN
+F 2 "" H 13900 10500 50  0001 C CNN
+F 3 "" H 13900 10500 50  0001 C CNN
+	1    13900 10500
+	-1   0    0    1
+$EndComp
+Wire Wire Line
+	13900 10500 13900 10300
+Wire Wire Line
+	13900 10100 14100 10100
+Wire Wire Line
+	14100 10200 13900 10200
+Connection ~ 13900 10200
+Wire Wire Line
+	13900 10200 13900 10100
+Wire Wire Line
+	14100 10300 13900 10300
+Connection ~ 13900 10300
+Wire Wire Line
+	13900 10300 13900 10200
+$Comp
+L power:+3.3V #PWR?
+U 1 1 5E8C53B5
+P 16200 10350
+F 0 "#PWR?" H 16200 10200 50  0001 C CNN
+F 1 "+3.3V" H 16215 10523 50  0000 C CNN
+F 2 "" H 16200 10350 50  0001 C CNN
+F 3 "" H 16200 10350 50  0001 C CNN
+	1    16200 10350
+	-1   0    0    1
+$EndComp
+Wire Wire Line
+	16100 10200 16200 10200
+Wire Wire Line
+	16200 10200 16200 10350
+$Comp
+L power:GND #PWR?
+U 1 1 5E8C8154
+P 13850 8800
+F 0 "#PWR?" H 13850 8550 50  0001 C CNN
+F 1 "GND" V 13855 8672 50  0000 R CNN
+F 2 "" H 13850 8800 50  0001 C CNN
+F 3 "" H 13850 8800 50  0001 C CNN
+	1    13850 8800
+	0    1    1    0
+$EndComp
+Wire Wire Line
+	14100 8600 13850 8600
+Wire Wire Line
+	13850 9000 14100 9000
+Wire Wire Line
+	14100 8900 13850 8900
+Connection ~ 13850 8900
+Wire Wire Line
+	13850 8900 13850 9000
+Wire Wire Line
+	14100 8800 13850 8800
+Wire Wire Line
+	13850 8600 13850 8700
+Connection ~ 13850 8800
+Wire Wire Line
+	13850 8800 13850 8900
+Wire Wire Line
+	14100 8700 13850 8700
+Connection ~ 13850 8700
+Wire Wire Line
+	13850 8700 13850 8800
 $EndSCHEMATC

Commit message: added motion
Other:
- moved on the sheet: LS1, R7
Changed lines of the file:
@@
 Wire Wire Line
 	1200 7350 1200 7300
-Text GLabel 6850 5950 2    50   Input ~ 0
-TX0
-Text GLabel 6850 6050 2    50   Input ~ 0
-RXI
 $Comp
 L power:+3.3V #PWR03
@@
 	10400 4250 10650 4250
 $Sheet
-S 9000 2450 1450 550
+S 9000 1950 1450 850
 U 5E70BD5E
 F0 "Sheet5E70BD5D" 50
 F1 "Sensor.sch" 50
-F2 "SCL" I R 10450 2600 50
-F3 "SDA" I R 10450 2700 50
-F4 "9_SDA" I R 10450 2800 50
-F5 "9_SCL" I R 10450 2900 50
-$EndSheet
-Wire Wire Line
-	10450 2700 10500 2700
-Wire Wire Line
-	10450 2600 10500 2600
-Text GLabel 10500 2700 2    50   Input ~ 0
+F2 "SCL" I R 10450 2100 50
+F3 "SDA" I R 10450 2200 50
+F4 "9_SDA" I R 10450 2300 50
+F5 "9_SCL" I R 10450 2400 50
+F6 "accel_cs" I L 9000 2000 50
+F7 "accel_scl" I L 9000 2100 50
+F8 "accel_sda" I L 9000 2200 50
+F9 "accel_sdo" I L 9000 2300 50
+F10 "BNO055_SCL" I L 9000 2400 50
+F11 "BNO055_SDA" I L 9000 2500 50
+F12 "BNO055_RESET" I L 9000 2600 50
+$EndSheet
+Wire Wire Line
+	10450 2200 10500 2200
+Wire Wire Line
+	10450 2100 10500 2100
+Text GLabel 10500 2200 2    50   Input ~ 0
 Pressure_SDA
-Text GLabel 10500 2600 2    50   Input ~ 0
+Text GLabel 10500 2100 2    50   Input ~ 0
 Pressure_SCL
 Wire Wire Line
@@
 NoConn ~ 1800 6850
 NoConn ~ 1800 6950
-Text GLabel 10550 2800 2    50   Input ~ 0
+Text GLabel 10550 2300 2    50   Input ~ 0
 9_SDA
-Text GLabel 10550 2900 2    50   Input ~ 0
+Text GLabel 10550 2400 2    50   Input ~ 0
 9_SCL
 Wire Wire Line
-	10450 2800 10550 2800
-Wire Wire Line
-	10450 2900 10550 2900
+	10450 2300 10550 2300
+Wire Wire Line
+	10450 2400 10550 2400
 Text GLabel 8250 950  2    50   Input ~ 0
 v_measure
@@
 L Mini_GPS_Tracker-rescue:CSS-J4D20-SMT-Sparkfun_Artemis-Mini_GPS_Tracker-rescue LS1
 U 1 1 5E7E01A2
-P 5500 3300
-F 0 "LS1" H 5605 3346 50  0000 L CNN
-F 1 "CSS-J4D20-SMT" H 5605 3255 50  0000 L CNN
-F 2 "Sparkfun-Artemis:CUI_CSS-J4D20-SMT" H 5500 3300 50  0001 L BNN
-F 3 "CUI" H 5500 3300 50  0001 L BNN
-F 4 "None" H 5500 3300 50  0001 L BNN "Field4"
-F 5 "CSS-J4D20-SMT" H 5500 3300 50  0001 L BNN "Field5"
-F 6 "Unavailable" H 5500 3300 50  0001 L BNN "Field6"
-F 7 "8.5 mm, 3.6 V, 90 dB, Surface Mount _SMT_, Magnetic Audio Transducer Buzzer" H 5500 3300 50  0001 L BNN "Field7"
-F 8 "None" H 5500 3300 50  0001 L BNN "Field8"
-	1    5500 3300
+P 2850 7050
+F 0 "LS1" H 2955 7096 50  0000 L CNN
+F 1 "CSS-J4D20-SMT" H 2955 7005 50  0000 L CNN
+F 2 "Sparkfun-Artemis:CUI_CSS-J4D20-SMT" H 2850 7050 50  0001 L BNN
+F 3 "CUI" H 2850 7050 50  0001 L BNN
+F 4 "None" H 2850 7050 50  0001 L BNN "Field4"
+F 5 "CSS-J4D20-SMT" H 2850 7050 50  0001 L BNN "Field5"
+F 6 "Unavailable" H 2850 7050 50  0001 L BNN "Field6"
+F 7 "8.5 mm, 3.6 V, 90 dB, Surface Mount _SMT_, Magnetic Audio Transducer Buzzer" H 2850 7050 50  0001 L BNN "Field7"
+F 8 "None" H 2850 7050 50  0001 L BNN "Field8"
+	1    2850 7050
 	1    0    0    -1
 $EndComp
@@
 L Device:R R7
 U 1 1 5E7E2738
-P 5500 2850
-F 0 "R7" H 5570 2896 50  0000 L CNN
-F 1 "0 ohm" H 5570 2805 50  0000 L CNN
-F 2 "Resistor_SMD:R_0805_2012Metric_Pad1.15x1.40mm_HandSolder" V 5430 2850 50  0001 C CNN
-F 3 "~" H 5500 2850 50  0001 C CNN
-	1    5500 2850
+P 2850 6600
+F 0 "R7" H 2920 6646 50  0000 L CNN
+F 1 "0 ohm" H 2920 6555 50  0000 L CNN
+F 2 "Resistor_SMD:R_0805_2012Metric_Pad1.15x1.40mm_HandSolder" V 2780 6600 50  0001 C CNN
+F 3 "~" H 2850 6600 50  0001 C CNN
+	1    2850 6600
 	1    0    0    -1
 $EndComp
@@
 L power:GND #PWR0116
 U 1 1 5E7E36E3
-P 5500 3600
-F 0 "#PWR0116" H 5500 3350 50  0001 C CNN
-F 1 "GND" H 5505 3427 50  0000 C CNN
-F 2 "" H 5500 3600 50  0001 C CNN
-F 3 "" H 5500 3600 50  0001 C CNN
-	1    5500 3600
+P 2850 7350
+F 0 "#PWR0116" H 2850 7100 50  0001 C CNN
+F 1 "GND" H 2855 7177 50  0000 C CNN
+F 2 "" H 2850 7350 50  0001 C CNN
+F 3 "" H 2850 7350 50  0001 C CNN
+	1    2850 7350
 	1    0    0    -1
 $EndComp
 Wire Wire Line
-	5500 3500 5500 3600
-Wire Wire Line
-	5500 3100 5500 3000
-Text GLabel 5500 2550 1    50   Input ~ 0
+	2850 7250 2850 7350
+Wire Wire Line
+	2850 6850 2850 6750
+Text GLabel 2850 6300 1    50   Input ~ 0
 buzzer
 Wire Wire Line
-	5500 2550 5500 2700
+	2850 6300 2850 6450
 Text GLabel 8250 3950 2    50   Input ~ 0
 buzzer

Commit message: added stm core connections
Parts:
- gave numbers to parts that had none: 1
Changed lines of the file:
@@
 	1    0    0    -1
 $EndComp
+Wire Wire Line
+	14100 8700 13850 8700
+Connection ~ 13850 8700
+Wire Wire Line
+	13850 8600 13850 8700
+Wire Wire Line
+	13850 8700 13850 8800
+Connection ~ 13850 8800
+Wire Wire Line
+	14100 8800 13850 8800
+Wire Wire Line
+	13850 8800 13850 8900
+Wire Wire Line
+	13850 8900 13850 9000
+Connection ~ 13850 8900
+Wire Wire Line
+	14100 8900 13850 8900
+Wire Wire Line
+	13850 9000 14100 9000
+Wire Wire Line
+	14100 8600 13850 8600
 $Comp
-L Sparkfun~Artemis:STM32H747XIH6 IC?
+L power:GND #PWR0130
+U 1 1 5E8C8154
+P 13850 8800
+F 0 "#PWR0130" H 13850 8550 50  0001 C CNN
+F 1 "GND" V 13855 8672 50  0000 R CNN
+F 2 "" H 13850 8800 50  0001 C CNN
+F 3 "" H 13850 8800 50  0001 C CNN
+	1    13850 8800
+	0    1    1    0
+$EndComp
+Wire Wire Line
+	16200 10200 16200 10350
+Wire Wire Line
+	16100 10200 16200 10200
+$Comp
+L power:+3.3V #PWR0131
+U 1 1 5E8C53B5
+P 16200 10350
+F 0 "#PWR0131" H 16200 10200 50  0001 C CNN
+F 1 "+3.3V" H 16215 10523 50  0000 C CNN
+F 2 "" H 16200 10350 50  0001 C CNN
+F 3 "" H 16200 10350 50  0001 C CNN
+	1    16200 10350
+	-1   0    0    1
+$EndComp
+Wire Wire Line
+	14100 10300 13900 10300
+Wire Wire Line
+	13900 10300 13900 10200
+Wire Wire Line
+	13900 10200 13900 10100
+Connection ~ 13900 10200
+Wire Wire Line
+	14100 10200 13900 10200
+Wire Wire Line
+	13900 10100 14100 10100
+Connection ~ 13900 10300
+Wire Wire Line
+	13900 10500 13900 10300
+$Comp
+L power:+3.3V #PWR0132
+U 1 1 5E8BD97D
+P 13900 10500
+F 0 "#PWR0132" H 13900 10350 50  0001 C CNN
+F 1 "+3.3V" H 13915 10673 50  0000 C CNN
+F 2 "" H 13900 10500 50  0001 C CNN
+F 3 "" H 13900 10500 50  0001 C CNN
+	1    13900 10500
+	-1   0    0    1
+$EndComp
+$Comp
+L Sparkfun~Artemis:STM32H747XIH6 IC1
 U 1 1 5E894707
 P 14100 -2900
-F 0 "IC?" H 15100 -2635 50  0000 C CNN
+F 0 "IC1" H 15100 -2635 50  0000 C CNN
 F 1 "STM32H747XIH6" H 15100 -2726 50  0000 C CNN
 F 2 "BGA265C80P17X17_1400X1400X110" H 15950 -2800 50  0001 L CNN
@@
 	1    0    0    -1
 $EndComp
-$Comp
-L power:+3.3V #PWR?
-U 1 1 5E8BD97D
-P 13900 10500
-F 0 "#PWR?" H 13900 10350 50  0001 C CNN
-F 1 "+3.3V" H 13915 10673 50  0000 C CNN
-F 2 "" H 13900 10500 50  0001 C CNN
-F 3 "" H 13900 10500 50  0001 C CNN
-	1    13900 10500
-	-1   0    0    1
-$EndComp
-Wire Wire Line
-	13900 10500 13900 10300
-Wire Wire Line
-	13900 10100 14100 10100
-Wire Wire Line
-	14100 10200 13900 10200
-Connection ~ 13900 10200
-Wire Wire Line
-	13900 10200 13900 10100
-Wire Wire Line
-	14100 10300 13900 10300
-Connection ~ 13900 10300
-Wire Wire Line
-	13900 10300 13900 10200
-$Comp
-L power:+3.3V #PWR?
-U 1 1 5E8C53B5
-P 16200 10350
-F 0 "#PWR?" H 16200 10200 50  0001 C CNN
-F 1 "+3.3V" H 16215 10523 50  0000 C CNN
-F 2 "" H 16200 10350 50  0001 C CNN
-F 3 "" H 16200 10350 50  0001 C CNN
-	1    16200 10350
-	-1   0    0    1
-$EndComp
-Wire Wire Line
-	16100 10200 16200 10200
-Wire Wire Line
-	16200 10200 16200 10350
-$Comp
-L power:GND #PWR?
-U 1 1 5E8C8154
-P 13850 8800
-F 0 "#PWR?" H 13850 8550 50  0001 C CNN
-F 1 "GND" V 13855 8672 50  0000 R CNN
-F 2 "" H 13850 8800 50  0001 C CNN
-F 3 "" H 13850 8800 50  0001 C CNN
-	1    13850 8800
-	0    1    1    0
-$EndComp
-Wire Wire Line
-	14100 8600 13850 8600
-Wire Wire Line
-	13850 9000 14100 9000
-Wire Wire Line
-	14100 8900 13850 8900
-Connection ~ 13850 8900
-Wire Wire Line
-	13850 8900 13850 9000
-Wire Wire Line
-	14100 8800 13850 8800
-Wire Wire Line
-	13850 8600 13850 8700
-Connection ~ 13850 8800
-Wire Wire Line
-	13850 8800 13850 8900
-Wire Wire Line
-	14100 8700 13850 8700
-Connection ~ 13850 8700
-Wire Wire Line
-	13850 8700 13850 8800
 $EndSCHEMATC

Commit message: updated core
Parts:
- removed IC1: STM32H747XIH6, BGA265C80P17X17_1400X1400X110, symbol Sparkfun~Artemis:STM32H747XIH6
- added U11: STM32F413ZHTx, Package_QFP:LQFP-144_20x20mm_P0.5mm, symbol MCU_ST_STM32F4:STM32F413ZHTx
Connections:
- wire segments 89 -> 72
Changed lines of the file:
@@
 	1    0    0    -1
 $EndComp
-Wire Wire Line
-	14100 8700 13850 8700
-Connection ~ 13850 8700
-Wire Wire Line
-	13850 8600 13850 8700
-Wire Wire Line
-	13850 8700 13850 8800
-Connection ~ 13850 8800
-Wire Wire Line
-	14100 8800 13850 8800
-Wire Wire Line
-	13850 8800 13850 8900
-Wire Wire Line
-	13850 8900 13850 9000
-Connection ~ 13850 8900
-Wire Wire Line
-	14100 8900 13850 8900
-Wire Wire Line
-	13850 9000 14100 9000
-Wire Wire Line
-	14100 8600 13850 8600
 $Comp
-L power:GND #PWR0130
-U 1 1 5E8C8154
-P 13850 8800
-F 0 "#PWR0130" H 13850 8550 50  0001 C CNN
-F 1 "GND" V 13855 8672 50  0000 R CNN
-F 2 "" H 13850 8800 50  0001 C CNN
-F 3 "" H 13850 8800 50  0001 C CNN
-	1    13850 8800
-	0    1    1    0
-$EndComp
-Wire Wire Line
-	16200 10200 16200 10350
-Wire Wire Line
-	16100 10200 16200 10200
-$Comp
-L power:+3.3V #PWR0131
-U 1 1 5E8C53B5
-P 16200 10350
-F 0 "#PWR0131" H 16200 10200 50  0001 C CNN
-F 1 "+3.3V" H 16215 10523 50  0000 C CNN
-F 2 "" H 16200 10350 50  0001 C CNN
-F 3 "" H 16200 10350 50  0001 C CNN
-	1    16200 10350
-	-1   0    0    1
-$EndComp
-Wire Wire Line
-	14100 10300 13900 10300
-Wire Wire Line
-	13900 10300 13900 10200
-Wire Wire Line
-	13900 10200 13900 10100
-Connection ~ 13900 10200
-Wire Wire Line
-	14100 10200 13900 10200
-Wire Wire Line
-	13900 10100 14100 10100
-Connection ~ 13900 10300
-Wire Wire Line
-	13900 10500 13900 10300
-$Comp
-L power:+3.3V #PWR0132
-U 1 1 5E8BD97D
-P 13900 10500
-F 0 "#PWR0132" H 13900 10350 50  0001 C CNN
-F 1 "+3.3V" H 13915 10673 50  0000 C CNN
-F 2 "" H 13900 10500 50  0001 C CNN
-F 3 "" H 13900 10500 50  0001 C CNN
-	1    13900 10500
-	-1   0    0    1
-$EndComp
-$Comp
-L Sparkfun~Artemis:STM32H747XIH6 IC1
-U 1 1 5E894707
-P 14100 -2900
-F 0 "IC1" H 15100 -2635 50  0000 C CNN
-F 1 "STM32H747XIH6" H 15100 -2726 50  0000 C CNN
-F 2 "BGA265C80P17X17_1400X1400X110" H 15950 -2800 50  0001 L CNN
-F 3 "https://www.st.com/en/microcontrollers-microprocessors/stm32h747xi.html" H 15950 -2900 50  0001 L CNN
-F 4 "ARM Microcontrollers - MCU" H 15950 -3000 50  0001 L CNN "Description"
-F 5 "1.1" H 15950 -3100 50  0001 L CNN "Height"
-F 6 "STMicroelectronics" H 15950 -3200 50  0001 L CNN "Manufacturer_Name"
-F 7 "STM32H747XIH6" H 15950 -3300 50  0001 L CNN "Manufacturer_Part_Number"
-F 8 "511-STM32H747XIH6" H 15950 -3400 50  0001 L CNN "Mouser Part Number"
-F 9 "https://www.mouser.com/Search/Refine.aspx?Keyword=511-STM32H747XIH6" H 15950 -3500 50  0001 L CNN "Mouser Price/Stock"
-F 10 "" H 15950 -3600 50  0001 L CNN "RS Part Number"
-F 11 "" H 15950 -3700 50  0001 L CNN "RS Price/Stock"
-	1    14100 -2900
+L MCU_ST_STM32F4:STM32F413ZHTx U11
+U 1 1 5E9BF2DA
+P 5950 -4100
+F 0 "U11" H 5950 -7789 50  0000 C CNN
+F 1 "STM32F413ZHTx" H 5950 -7880 50  0000 C CNN
+F 2 "Package_QFP:LQFP-144_20x20mm_P0.5mm" H 4950 -7500 50  0001 R CNN
+F 3 "http://www.st.com/st-web-ui/static/active/en/resource/technical/document/datasheet/DM00282249.pdf" H 5950 -4100 50  0001 C CNN
+	1    5950 -4100
 	1    0    0    -1
 $EndComp

Commit message: added back usb driver chip
Parts:
- added U?: FT230XS, Package_SO:SSOP-16_3.9x4.9mm_P0.635mm, symbol Interface_USB:FT230XS
Changed lines of the file:
@@
+	1    0    0    -1
+$EndComp
+$Comp
+L Interface_USB:FT230XS U?
+U 1 1 5E9B8EAD
+P 3600 5200
+F 0 "U?" H 3600 6081 50  0000 C CNN
+F 1 "FT230XS" H 3600 5990 50  0000 C CNN
+F 2 "Package_SO:SSOP-16_3.9x4.9mm_P0.635mm" H 4600 4600 50  0001 C CNN
+F 3 "https://www.ftdichip.com/Support/Documents/DataSheets/ICs/DS_FT230X.pdf" H 3600 5200 50  0001 C CNN
+	1    3600 5200
 	1    0    0    -1
 $EndComp

Commit message: added back usb circuit
Parts:
- added C?: 100nF, symbol pspice:CAP
Connections:
- wire segments 72 -> 91
Other:
- moved on the sheet: LS1, R7, U?
Changed lines of the file:
@@
 L Mini_GPS_Tracker-rescue:CSS-J4D20-SMT-Sparkfun_Artemis-Mini_GPS_Tracker-rescue LS1
 U 1 1 5E7E01A2
-P 2850 7050
-F 0 "LS1" H 2955 7096 50  0000 L CNN
-F 1 "CSS-J4D20-SMT" H 2955 7005 50  0000 L CNN
-F 2 "Sparkfun-Artemis:CUI_CSS-J4D20-SMT" H 2850 7050 50  0001 L BNN
-F 3 "CUI" H 2850 7050 50  0001 L BNN
-F 4 "None" H 2850 7050 50  0001 L BNN "Field4"
-F 5 "CSS-J4D20-SMT" H 2850 7050 50  0001 L BNN "Field5"
-F 6 "Unavailable" H 2850 7050 50  0001 L BNN "Field6"
-F 7 "8.5 mm, 3.6 V, 90 dB, Surface Mount _SMT_, Magnetic Audio Transducer Buzzer" H 2850 7050 50  0001 L BNN "Field7"
-F 8 "None" H 2850 7050 50  0001 L BNN "Field8"
-	1    2850 7050
+P 6250 5400
+F 0 "LS1" H 6355 5446 50  0000 L CNN
+F 1 "CSS-J4D20-SMT" H 6355 5355 50  0000 L CNN
+F 2 "Sparkfun-Artemis:CUI_CSS-J4D20-SMT" H 6250 5400 50  0001 L BNN
+F 3 "CUI" H 6250 5400 50  0001 L BNN
+F 4 "None" H 6250 5400 50  0001 L BNN "Field4"
+F 5 "CSS-J4D20-SMT" H 6250 5400 50  0001 L BNN "Field5"
+F 6 "Unavailable" H 6250 5400 50  0001 L BNN "Field6"
+F 7 "8.5 mm, 3.6 V, 90 dB, Surface Mount _SMT_, Magnetic Audio Transducer Buzzer" H 6250 5400 50  0001 L BNN "Field7"
+F 8 "None" H 6250 5400 50  0001 L BNN "Field8"
+	1    6250 5400
 	1    0    0    -1
 $EndComp
@@
 L Device:R R7
 U 1 1 5E7E2738
-P 2850 6600
-F 0 "R7" H 2920 6646 50  0000 L CNN
-F 1 "0 ohm" H 2920 6555 50  0000 L CNN
-F 2 "Resistor_SMD:R_0805_2012Metric_Pad1.15x1.40mm_HandSolder" V 2780 6600 50  0001 C CNN
-F 3 "~" H 2850 6600 50  0001 C CNN
-	1    2850 6600
+P 6250 4950
+F 0 "R7" H 6320 4996 50  0000 L CNN
+F 1 "0 ohm" H 6320 4905 50  0000 L CNN
+F 2 "Resistor_SMD:R_0805_2012Metric_Pad1.15x1.40mm_HandSolder" V 6180 4950 50  0001 C CNN
+F 3 "~" H 6250 4950 50  0001 C CNN
+	1    6250 4950
 	1    0    0    -1
 $EndComp
@@
 L power:GND #PWR0116
 U 1 1 5E7E36E3
-P 2850 7350
-F 0 "#PWR0116" H 2850 7100 50  0001 C CNN
-F 1 "GND" H 2855 7177 50  0000 C CNN
-F 2 "" H 2850 7350 50  0001 C CNN
-F 3 "" H 2850 7350 50  0001 C CNN
-	1    2850 7350
-	1    0    0    -1
-$EndComp
-Wire Wire Line
-	2850 7250 2850 7350
-Wire Wire Line
-	2850 6850 2850 6750
-Text GLabel 2850 6300 1    50   Input ~ 0
+P 6250 5700
+F 0 "#PWR0116" H 6250 5450 50  0001 C CNN
+F 1 "GND" H 6255 5527 50  0000 C CNN
+F 2 "" H 6250 5700 50  0001 C CNN
+F 3 "" H 6250 5700 50  0001 C CNN
+	1    6250 5700
+	1    0    0    -1
+$EndComp
+Wire Wire Line
+	6250 5600 6250 5700
+Wire Wire Line
+	6250 5200 6250 5100
+Text GLabel 6250 4650 1    50   Input ~ 0
 buzzer
 Wire Wire Line
-	2850 6300 2850 6450
+	6250 4650 6250 4800
 Text GLabel 8250 3950 2    50   Input ~ 0
 buzzer
@@
 L Interface_USB:FT230XS U?
 U 1 1 5E9B8EAD
-P 3600 5200
-F 0 "U?" H 3600 6081 50  0000 C CNN
-F 1 "FT230XS" H 3600 5990 50  0000 C CNN
-F 2 "Package_SO:SSOP-16_3.9x4.9mm_P0.635mm" H 4600 4600 50  0001 C CNN
-F 3 "https://www.ftdichip.com/Support/Documents/DataSheets/ICs/DS_FT230X.pdf" H 3600 5200 50  0001 C CNN
-	1    3600 5200
-	1    0    0    -1
-$EndComp
+P 3500 5250
+F 0 "U?" H 3500 6131 50  0000 C CNN
+F 1 "FT230XS" H 3500 6040 50  0000 C CNN
+F 2 "Package_SO:SSOP-16_3.9x4.9mm_P0.635mm" H 4500 4650 50  0001 C CNN
+F 3 "https://www.ftdichip.com/Support/Documents/DataSheets/ICs/DS_FT230X.pdf" H 3500 5250 50  0001 C CNN
+	1    3500 5250
+	1    0    0    -1
+$EndComp
+Wire Wire Line
+	1800 5150 2800 5150
+Wire Wire Line
+	1800 5250 2800 5250
+$Comp
+L power:GND #PWR?
+U 1 1 5E9DAEFA
+P 3500 6100
+F 0 "#PWR?" H 3500 5850 50  0001 C CNN
+F 1 "GND" H 3505 5927 50  0000 C CNN
+F 2 "" H 3500 6100 50  0001 C CNN
+F 3 "" H 3500 6100 50  0001 C CNN
+	1    3500 6100
+	1    0    0    -1
+$EndComp
+Wire Wire Line
+	3400 5950 3400 6100
+Wire Wire Line
+	3400 6100 3500 6100
+Wire Wire Line
+	3500 6100 3600 6100
+Wire Wire Line
+	3600 6100 3600 5950
+Connection ~ 3500 6100
+Text GLabel 4350 5050 2    50   Input ~ 0
+RTS
+Wire Wire Line
+	4200 5050 4350 5050
+Text GLabel 4550 4950 2    50   Input ~ 0
+RXI
+Text GLabel 4550 4850 2    50   Input ~ 0
+TX0
+Wire Wire Line
+	4200 4850 4550 4850
+Wire Wire Line
+	4200 4950 4550 4950
+$Comp
+L power:+3.3V #PWR?
+U 1 1 5E9E8361
+P 3400 4350
+F 0 "#PWR?" H 3400 4200 50  0001 C CNN
+F 1 "+3.3V" H 3415 4523 50  0000 C CNN
+F 2 "" H 3400 4350 50  0001 C CNN
+F 3 "" H 3400 4350 50  0001 C CNN
+	1    3400 4350
+	1    0    0    -1
+$EndComp
+Wire Wire Line
+	3400 4550 3400 4350
+$Comp
+L pspice:CAP C?
+U 1 1 5E9EBAC9
+P 4000 4400
+F 0 "C?" V 3685 4400 50  0000 C CNN
+F 1 "100nF" V 3776 4400 50  0000 C CNN
+F 2 "" H 4000 4400 50  0001 C CNN
+F 3 "~" H 4000 4400 50  0001 C CNN
+	1    4000 4400
+	0    1    1    0
+$EndComp
+$Comp
+L power:GND #PWR?
+U 1 1 5E9EC72D
+P 4400 4400
+F 0 "#PWR?" H 4400 4150 50  0001 C CNN
+F 1 "GND" V 4405 4272 50  0000 R CNN
+F 2 "" H 4400 4400 50  0001 C CNN
+F 3 "" H 4400 4400 50  0001 C CNN
+	1    4400 4400
+	0    -1   -1   0
+$EndComp
+Wire Wire Line
+	4250 4400 4400 4400
+Wire Wire Line
+	2800 5450 2550 5450
+Wire Wire Line
+	2550 5450 2550 4850
+Wire Wire Line
+	2550 3950 3600 3950
+Wire Wire Line
+	3600 3950 3600 4400
+Wire Wire Line
+	3750 4400 3600 4400
+Connection ~ 3600 4400
+Wire Wire Line
+	3600 4400 3600 4550
+Wire Wire Line
+	2800 4850 2550 4850
+Connection ~ 2550 4850
+Wire Wire Line
+	2550 4850 2550 3950
 $EndSCHEMATC
