File: Mini_GPS_Tracker/Accel.sch (KiCad schematic (older format))
At the start: 1 part

Commit message: Add files via upload
Making update for 100 pin CPU
Parts:
- gave numbers to parts that had none: 1
Changed lines of the file:
@@
 EESchema Schematic File Version 4
+LIBS:Mini_GPS_Tracker-cache
 EELAYER 30 0
 EELAYER END
 $Descr A4 11693 8268
 encoding utf-8
-Sheet 10 11
+Sheet 10 8
 Title ""
 Date ""
@@
 	7850 4150 7750 4150
 $Comp
-L SamacSys_Parts:ADXL375BCCZ IC?
+L SamacSys_Parts:ADXL375BCCZ IC1
 U 1 1 5EA14D39
 P 5750 4150
-F 0 "IC?" H 6750 5131 50  0000 C CNN
+F 0 "IC1" H 6750 5131 50  0000 C CNN
 F 1 "ADXL375BCCZ" H 6750 5040 50  0000 C CNN
 F 2 "CC-14-1" H 7600 4750 50  0001 L CNN
@@
 	5550 4450 5550 4550
 $Comp
-L power:GND #PWR?
+L power:GND #PWR010
 U 1 1 5EA15CA9
 P 5400 4450
-F 0 "#PWR?" H 5400 4200 50  0001 C CNN
+F 0 "#PWR010" H 5400 4200 50  0001 C CNN
 F 1 "GND" H 5405 4277 50  0000 C CNN
 F 2 "" H 5400 4450 50  0001 C CNN
@@
 	4800 4650 5750 4650
 $Comp
-L power:+3.3V #PWR?
+L power:+3.3V #PWR06
 U 1 1 5EA1659C
 P 5100 4150
-F 0 "#PWR?" H 5100 4000 50  0001 C CNN
+F 0 "#PWR06" H 5100 4000 50  0001 C CNN
 F 1 "+3.3V" H 5115 4323 50  0000 C CNN
 F 2 "" H 5100 4150 50  0001 C CNN
