File: Mini_GPS_Tracker.kicad_pcb (KiCad board)
At the start: 4 copper layers, 38.1 x 105.4 mm, 56 parts, among them J1 USB_C_Receptacle, J2 Screw_Terminal_01x02, J3 901-10512-1, J4 Conn_ARM_JTAG_SWD_10, SW1 SW_Push, SW2 MLL1200S, U1 FT230XS, U2 MS5611-01BA, U3 LD1117S33TR_SOT223, U4 MAX-8Q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

Commit message: Add files via upload
Ground pour
Routing:
- added copper zone on GND, net GND
Changed lines of the file:
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@@
   (page A4)
   (layers
-    (0 F.Cu signal)
+    (0 F.Cu signal hide)
     (1 GND power)
-    (2 PWR power)
-    (31 B.Cu signal)
+    (2 PWR power hide)
+    (31 B.Cu signal hide)
     (32 B.Adhes user hide)
     (33 F.Adhes user)
@@
   (segment (start 153.67 38.1) (end 156.21 35.56) (width 0.25) (layer F.Cu) (net 0))
   (segment (start 156.21 35.56) (end 166.37 35.56) (width 0.25) (layer F.Cu) (net 0))
-  (via (at 161.29 121.92) (size 0.8) (drill 0.4) (layers F.Cu B.Cu) (net 8))
-  (via (at 149.86 124.46) (size 0.8) (drill 0.4) (layers F.Cu B.Cu) (net 138))
-  (via (at 161.29 127) (size 0.8) (drill 0.4) (layers F.Cu B.Cu) (net 138))
-  (via (at 179.07 81.28) (size 0.8) (drill 0.4) (layers F.Cu B.Cu) (net 3))
-  (via (at 180.34 83.82) (size 0.8) (drill 0.4) (layers F.Cu B.Cu) (net 3))
-  (via (at 172.72 87.63) (size 0.8) (drill 0.4) (layers F.Cu B.Cu) (net 3))
-  (via (at 171.45 91.44) (size 0.8) (drill 0.4) (layers F.Cu B.Cu) (net 101))
   (segment (start 181.728 106.107) (end 181.728 106.807) (width 0.25) (layer F.Cu) (net 1) (status 30))
   (segment (start 181.728 106.807) (end 181.728 107.043) (width 0.25) (layer F.Cu) (net 1) (status 30))
@@
   (segment (start 157.796 132.145) (end 159.7 132.145) (width 0.25) (layer GND) (net 2))
   (segment (start 157.48 132.461) (end 157.796 132.145) (width 0.25) (layer GND) (net 2))
+  (via (at 179.07 81.28) (size 0.8) (drill 0.4) (layers F.Cu B.Cu) (net 3))
+  (via (at 180.34 83.82) (size 0.8) (drill 0.4) (layers F.Cu B.Cu) (net 3))
+  (via (at 172.72 87.63) (size 0.8) (drill 0.4) (layers F.Cu B.Cu) (net 3))
   (segment (start 154.187 69.351) (end 154.178 69.342) (width 0.25) (layer F.Cu) (net 3) (status 30))
   (segment (start 166.379 118.237) (end 166.379 118.346) (width 0.25) (layer F.Cu) (net 3) (status 30))
@@
   (segment (start 176.784 90.678) (end 178.435 92.329) (width 0.203) (layer GND) (net 3))
   (segment (start 176.784 90.043) (end 176.784 90.678) (width 0.203) (layer GND) (net 3))
-  (segment (start 169.665 84.709) (end 169.418 84.709) (width 0.203) (layer F.Cu) (net 122))
-  (segment (start 169.418 84.709) (end 169.418 84.709) (width 0.203) (layer F.Cu) (net 122))
   (segment (start 158.877 84.709) (end 152.4 78.232) (width 0.203) (layer GND) (net 3))
   (segment (start 152.4 78.232) (end 152.146 77.978) (width 0.203) (layer GND) (net 3))
@@
   (segment (start 161.052585 119.278585) (end 164.329 122.555) (width 0.25) (layer F.Cu) (net 7))
   (segment (start 161.052585 119.142585) (end 161.052585 119.278585) (width 0.25) (layer F.Cu) (net 7))
+  (via (at 161.29 121.92) (size 0.8) (drill 0.4) (layers F.Cu B.Cu) (net 8))
   (via (at 166.624 101.6) (size 0.8) (drill 0.4) (layers F.Cu B.Cu) (net 8))
   (via (at 162.56 119.38) (size 0.8) (drill 0.4) (layers F.Cu B.Cu) (net 8))
@@
   (segment (start 151.706 79.652298) (end 151.26049 79.206788) (width 0.203) (layer F.Cu) (net 100))
   (segment (start 151.706 80.055) (end 151.706 79.652298) (width 0.203) (layer F.Cu) (net 100))
+  (via (at 171.45 91.44) (size 0.8) (drill 0.4) (layers F.Cu B.Cu) (net 101))
   (segment (start 165.31 93.147) (end 165.21 93.147) (width 0.203) (layer F.Cu) (net 101))
   (segment (start 165.21 93.147) (end 165.21 92.312) (width 0.203) (layer F.Cu) (net 101))
@@
   (segment (start 149.252499 103.100279) (end 149.252499 103.278499) (width 0.203) (layer F.Cu) (net 121))
   (segment (start 154.949 100.711) (end 154.453956 100.711) (width 0.203) (layer F.Cu) (net 121))
+  (segment (start 169.665 84.709) (end 169.418 84.709) (width 0.203) (layer F.Cu) (net 122))
+  (segment (start 169.418 84.709) (end 169.418 84.709) (width 0.203) (layer F.Cu) (net 122))
   (segment (start 176.23832 130.001) (end 176.69932 129.54) (width 0.25) (layer F.Cu) (net 123))
   (segment (start 174.117 130.001) (end 176.23832 130.001) (width 0.25) (layer F.Cu) (net 123))
@@
   (segment (start 172.61 93.147) (end 172.51 93.147) (width 0.25) (layer F.Cu) (net 131) (status 30))
   (segment (start 165.21 95.147) (end 165.31 95.147) (width 0.25) (layer F.Cu) (net 133) (status 30))
+  (via (at 149.86 124.46) (size 0.8) (drill 0.4) (layers F.Cu B.Cu) (net 138))
+  (via (at 161.29 127) (size 0.8) (drill 0.4) (layers F.Cu B.Cu) (net 138))
   (segment (start 151.145 124.7775) (end 149.86 126.0625) (width 0.25) (layer F.Cu) (net 138))
   (segment (start 153.61 124.7775) (end 151.145 124.7775) (width 0.25) (layer F.Cu) (net 138))
@@
       )
     )
+  )
+  (zone (net 2) (net_name GND) (layer GND) (hatch edge 0.508)
+    (connect_pads (clearance 0.508))
+    (min_thickness 0.254)
+    (fill yes (arc_segments 32) (thermal_gap 0.508) (thermal_bridge_width 0.508))
+    (polygon
+      (pts
+        (xy 147.32 34.29) (xy 184.15 34.29) (xy 185.42 139.7) (xy 147.32 139.7)
+      )
+    )
